Commit message: Solved Spawn Issues

File: car_robot/urdf/car_robot.urdf.xacro (robot description, xacro)
@@ -5,23 +5,34 @@
 <robot
   name="car_robot" xmlns:xacro="http://ros.org/wiki/xacro">
-  <!-- <ros2_control name="GazeboSystem" type="system">
- <hardware>
-     <plugin>gazebo_ros2_control/GazeboSystem</plugin>
- </hardware> -->
+  <xacro:macro name="body_color">
+    <visual>
+    <material>
+        <ambient>0.8 0.558823529411765 0.1 1</ambient>
+        <diffuse>0.8 0.558823529411765 0.1 1</diffuse>
+        <specular>0.1 0.1 0.1 1</specular>
+        <emissive>0 0 0 0</emissive>
+    </material>
+    </visual>
+</xacro:macro>
+<gazebo reference="base_link">
+    <xacro:body_color />
+</gazebo>
+  # Add this before base link
+<link name="dummy_link"></link>
   <link
     name="base_link">
     <inertial>
       <origin
-        xyz="0.0102934841398985 -0.00376231068740884 5.43044143984843E-17"
-        rpy="0 0 0" />
-      <mass
-        value="25.6200869444948" />
-      <inertia
-        ixx="0.571525055680453"
-        ixy="0.0234910482197784"
-        ixz="-1.97435940527347E-16"
-        iyy="2.52764338096436"
-        iyz="-2.99012692149574E-17"
-        izz="1.99201719065782" />
+        xyz="-0.00677096096599195 -7.40324226081856E-09 0.306370957352742"
+        rpy="0 0 0" />
+      <mass
+        value="40.1297473551325" />
+      <inertia
+        ixx="1.26922453974044"
+        ixy="1.04912166627978E-07"
+        ixz="-0.0347492884684778"
+        iyy="3.34453299992272"
+        iyz="1.64404574479948E-08"
+        izz="4.11157029873108" />
     </inertial>
     <visual>
@@ -36,4 +47,166 @@
         name="">
         <color
+          rgba="0.752941176470588 0.752941176470588 0.752941176470588 1" />
+      </material>
+    </visual>
+    <collision>
+      <origin
+        xyz="0 0 0"
+        rpy="0 0 0" />
+      <geometry>
+        <mesh
+          filename="package://car_robot/meshes/base_link.STL" />
+      </geometry>
+    </collision>
+  </link>
+  # Add this after base link
+<joint name="dummy_joint" type="fixed">
+    <origin rpy="0 0 0" xyz="0 0 0" />
+    <parent link="dummy_link"/>
+    <child link="base_link"/>
+</joint>
+  <link
+    name="front-left-hinge">
+    <inertial>
+      <origin
+        xyz="3.88578058618805E-16 -6.10622663543836E-16 -0.118799628145585"
+        rpy="0 0 0" />
+      <mass
+        value="0.633612488698204" />
+      <inertia
+        ixx="0.00419900401400481"
+        ixy="0.000173645794203951"
+        ixz="-1.07917330807736E-18"
+        iyy="0.00247709562888137"
+        iyz="-1.52690795674631E-18"
+        izz="0.00202629416547586" />
+    </inertial>
+    <visual>
+      <origin
+        xyz="0 0 0"
+        rpy="0 0 0" />
+      <geometry>
+        <mesh
+          filename="package://car_robot/meshes/front-left-hinge.STL" />
+      </geometry>
+      <material
+        name="">
+        <color
+          rgba="1 1 0 1" />
+      </material>
+    </visual>
+    <collision>
+      <origin
+        xyz="0 0 0"
+        rpy="0 0 0" />
+      <geometry>
+        <mesh
+          filename="package://car_robot/meshes/front-left-hinge.STL" />
+      </geometry>
+    </collision>
+  </link>
+  <joint
+    name="fl-hinge"
+    type="revolute">
+    <origin
+      xyz="0.254 0.1397 0.3021"
+      rpy="0 0 -3.1416" />
+    <parent
+      link="base_link" />
+    <child
+      link="front-left-hinge" />
+    <axis
+      xyz="0 0 -1" />
+    <limit
+      lower="0"
+      upper="0"
+      effort="0"
+      velocity="0" />
+  </joint>
+  <link
+    name="front-left-wheeel">
+    <inertial>
+      <origin
+        xyz="-0.00757015271891448 2.77555756156289E-17 -0.0758230359970678"
+        rpy="0 0 0" />
+      <mass
+        value="2.43249992415545" />
+      <inertia
+        ixx="0.00760381168766053"
+        ixy="-8.24720643585744E-19"
+        ixz="0.00051389219741489"
+        iyy="0.00755250482076537"
+        iyz="-3.62054828260286E-19"
+        izz="0.0126996752980334" />
+    </inertial>
+    <visual>
+      <origin
+        xyz="0 0 0"
+        rpy="0 0 0" />
+      <geometry>
+        <mesh
+          filename="package://car_robot/meshes/front-left-wheeel.STL" />
+      </geometry>
+      <material
+        name="">
+        <color
+          rgba="0 0 0 1" />
+      </material>
+    </visual>
+    <collision>
+      <origin
+        xyz="0 0 0"
+        rpy="0 0 0" />
+      <geometry>
+        <mesh
+          filename="package://car_robot/meshes/front-left-wheeel.STL" />
+      </geometry>
+    </collision>
+  </link>
+  <joint
+    name="fl-wheel"
+    type="revolute">
+    <origin
+      xyz="0.0075702 -0.075823 -0.2005"
+      rpy="1.5708 0 0" />
+    <parent
+      link="front-left-hinge" />
+    <child
+      link="front-left-wheeel" />
+    <axis
+      xyz="0.099346 0 0.99505" />
+    <limit
+      lower="0"
+      upper="0"
+      effort="0"
+      velocity="0" />
+  </joint>
+  <link
+    name="front-left-axle">
+    <inertial>
+      <origin
+        xyz="-0.00757015271891331 -2.77555756156289E-17 -0.0758230359970657"
+        rpy="0 0 0" />
+      <mass
+        value="0.0772222198144586" />
+      <inertia
+        ixx="0.000151131456795402"
+        ixy="-2.82674264757069E-21"
+        ixz="-1.44671657852651E-05"
+        iyy="0.000152575854964957"
+        iyz="-2.83127986289767E-20"
+        izz="7.67198408649241E-06" />
+    </inertial>
+    <visual>
+      <origin
+        xyz="0 0 0"
+        rpy="0 0 0" />
+      <geometry>
+        <mesh
+          filename="package://car_robot/meshes/front-left-axle.STL" />
+      </geometry>
+      <material
+        name="">
+        <color
           rgba="0.792156862745098 0.819607843137255 0.933333333333333 1" />
       </material>
@@ -45,31 +218,165 @@
       <geometry>
         <mesh
-          filename="package://car_robot/meshes/base_link.STL" />
-      </geometry>
-    </collision>
-  </link>
-  <link
-    name="left-hinge">
-    <inertial>
-      <origin
-        xyz="-2.77555756156289E-17 3.33066907387547E-16 -0.0846241805160345"
-        rpy="0 0 0" />
-      <mass
-        value="0.62854541390723" />
-      <inertia
-        ixx="0.00235146189900645"
-        ixy="-2.71050543121376E-19"
-        ixz="3.28576308435801E-19"
-        iyy="0.00410804378839769"
-        iyz="5.90295081884936E-18"
-        izz="0.00202588553122934" />
-    </inertial>
-    <visual>
-      <origin
-        xyz="0 0 0"
-        rpy="0 0 0" />
-      <geometry>
-        <mesh
-          filename="package://car_robot/meshes/left-hinge.STL" />
+          filename="package://car_robot/meshes/front-left-axle.STL" />
+      </geometry>
+    </collision>
+  </link>
+  <joint
+    name="fl-axle"
+    type="revolute">
+    <origin
+      xyz="0.0075702 -0.075823 -0.2005"
+      rpy="1.5708 0 0" />
+    <parent
+      link="front-left-hinge" />
+    <child
+      link="front-left-axle" />
+    <axis
+      xyz="0.099346 0 0.99505" />
+    <limit
+      lower="0"
+      upper="0"
+      effort="0"
+      velocity="0" />
+  </joint>
+  <link
+    name="front-right-hinge">
+    <inertial>
+      <origin
+        xyz="-5.55111512312578E-17 -8.32667268468867E-17 -0.118799628145586"
+        rpy="0 0 0" />
+      <mass
+        value="0.633612488698204" />
+      <inertia
+        ixx="0.00392482649211829"
+        ixy="0.000653519794869028"
+        ixz="-1.24551730795087E-19"
+        iyy="0.0027512731507679"
+        iyz="-4.19591111294197E-19"
+        izz="0.00202629416547586" />
+    </inertial>
+    <visual>
+      <origin
+        xyz="0 0 0"
+        rpy="0 0 0" />
+      <geometry>
+        <mesh
+          filename="package://car_robot/meshes/front-right-hinge.STL" />
+      </geometry>
+      <material
+        name="">
+        <color
+          rgba="1 1 0 1" />
+      </material>
+    </visual>
+    <collision>
+      <origin
+        xyz="0 0 0"
+        rpy="0 0 0" />
+      <geometry>
+        <mesh
+          filename="package://car_robot/meshes/front-right-hinge.STL" />
+      </geometry>
+    </collision>
+  </link>
+  <joint
+    name="fr-hinge"
+    type="revolute">
+    <origin
+      xyz="0.254 -0.1397 0.3021"
+      rpy="0 0 -3.1416" />
+    <parent
+      link="base_link" />
+    <child
+      link="front-right-hinge" />
+    <axis
+      xyz="0 0 -1" />
+    <limit
+      lower="0"
+      upper="0"
+      effort="0"
+      velocity="0" />
+  </joint>
+  <link
+    name="front-right-wheel">
+    <inertial>
+      <origin
+        xyz="-0.031042070676579 8.32667268468867E-17 -0.0695904436550727"
+        rpy="0 0 0" />
+      <mass
+        value="2.43249992415545" />
+      <inertia
+        ixx="0.0084152202786371"
+        ixy="-2.50693797234352E-18"
+        ixz="0.00193404467398112"
+        iyy="0.00755250482076537"
+        iyz="-3.20124118023232E-18"
+        izz="0.0118882667070568" />
+    </inertial>
+    <visual>
+      <origin
+        xyz="0 0 0"
+        rpy="0 0 0" />
+      <geometry>
+        <mesh
+          filename="package://car_robot/meshes/front-right-wheel.STL" />
+      </geometry>
+      <material
+        name="">
+        <color
+          rgba="0 0 0 1" />
+      </material>
+    </visual>
+    <collision>
+      <origin
+        xyz="0 0 0"
+        rpy="0 0 0" />
+      <geometry>
+        <mesh
+          filename="package://car_robot/meshes/front-right-wheel.STL" />
+      </geometry>
+    </collision>
+  </link>
+  <joint
+    name="fr-wheel"
+    type="revolute">
+    <origin
+      xyz="-0.031042 0.06959 -0.2005"
+      rpy="1.5708 0 3.1416" />
+    <parent
+      link="front-right-hinge" />
+    <child
+      link="front-right-wheel" />
+    <axis
+      xyz="-0.40738 0 -0.91326" />
+    <limit
+      lower="0"
+      upper="0"
+      effort="0"
+      velocity="0" />
+  </joint>
+  <link
+    name="front-right-axle">
+    <inertial>
+      <origin
+        xyz="-0.0310420706765801 8.32667268468867E-17 -0.0695904436550753"
+        rpy="0 0 0" />
+      <mass
+        value="0.0772222198144586" />
+      <inertia
+        ixx="0.000128288567441763"
+        ixy="3.72486511718043E-20"
+        ixz="-5.44474990578691E-05"
+        iyy="0.000152575854964957"
+        iyz="8.14822018357058E-20"
+        izz="3.05148734401304E-05" />
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
Commit message: Solved Teleop Issue

File: car_robot/urdf/car_robot.urdf.xacro (robot description, xacro)
@@ -18,11 +18,9 @@
     <xacro:body_color />
 </gazebo>
-  # Add this before base link
-<link name="dummy_link"></link>
   <link
     name="base_link">
     <inertial>
       <origin
-        xyz="-0.00677096096599195 -7.40324226081856E-09 0.306370957352742"
+        xyz="-0.00677096096599197 -7.40324229928916E-09 0.0650709573527417"
         rpy="0 0 0" />
       <mass
@@ -30,8 +28,8 @@
       <inertia
         ixx="1.26922453974044"
-        ixy="1.04912166627978E-07"
+        ixy="1.04912166639753E-07"
         ixz="-0.0347492884684778"
         iyy="3.34453299992272"
-        iyz="1.64404574479948E-08"
+        iyz="1.6440457327724E-08"
         izz="4.11157029873108" />
     </inertial>
@@ -60,24 +58,18 @@
     </collision>
   </link>
-  # Add this after base link
-<joint name="dummy_joint" type="fixed">
-    <origin rpy="0 0 0" xyz="0 0 0" />
-    <parent link="dummy_link"/>
-    <child link="base_link"/>
-</joint>
   <link
     name="front-left-hinge">
     <inertial>
       <origin
-        xyz="3.88578058618805E-16 -6.10622663543836E-16 -0.118799628145585"
+        xyz="0 2.77555756156289E-17 -0.118799628145585"
         rpy="0 0 0" />
       <mass
         value="0.633612488698204" />
       <inertia
-        ixx="0.00419900401400481"
-        ixy="0.000173645794203951"
-        ixz="-1.07917330807736E-18"
-        iyy="0.00247709562888137"
-        iyz="-1.52690795674631E-18"
+        ixx="0.0042046227153009"
+        ixy="-0.000142990919869844"
+        ixz="-1.30495243379754E-18"
+        iyy="0.00247147692758528"
+        iyz="-6.30427138270604E-19"
         izz="0.00202629416547586" />
     </inertial>
@@ -108,7 +100,7 @@
   <joint
     name="fl-hinge"
-    type="revolute">
-    <origin
-      xyz="0.254 0.1397 0.3021"
+    type="continuous">
+    <origin
+      xyz="0.254 0.1397 0.0608"
       rpy="0 0 -3.1416" />
     <parent
@@ -118,4 +110,62 @@
     <axis
       xyz="0 0 -1" />
+    <limit
+      lower="-0.69"
+      upper="0.69"
+      effort="0"
+      velocity="0" />
+  </joint>
+  <link
+    name="front-left-wheeel">
+    <inertial>
+      <origin
+        xyz="0.00622369727134658 -2.77555756156289E-16 -0.0759454119237928"
+        rpy="0 0 0" />
+      <mass
+        value="2.43249992415545" />
+      <inertia
+        ixx="0.00758718354662836"
+        ixy="-1.26731196831282E-18"
+        ixz="-0.000423171308923178"
+        iyy="0.00755250482076537"
+        iyz="-1.68232117058127E-19"
+        izz="0.0127163034390655" />
+    </inertial>
+    <visual>
+      <origin
+        xyz="0 0 0"
+        rpy="0 0 0" />
+      <geometry>
+        <mesh
+          filename="package://car_robot/meshes/front-left-wheeel.STL" />
+      </geometry>
+      <material
+        name="">
+        <color
+          rgba="0 0 0 1" />
+      </material>
+    </visual>
+    <collision>
+      <origin
+        xyz="0 0 0"
+        rpy="0 0 0" />
+      <geometry>
+        <mesh
+          filename="package://car_robot/meshes/front-left-wheeel.STL" />
+      </geometry>
+    </collision>
+  </link>
+  <joint
+    name="fl-wheel"
+    type="continuous">
+    <origin
+      xyz="-0.00622369727134681 -0.0759454119237924 -0.2005"
+      rpy="1.5707963267949 0 0" />
+    <parent
+      link="front-left-hinge" />
+    <child
+      link="front-left-wheeel" />
+    <axis
+      xyz="-0.0816758172092811 0 0.996658949131144" />
     <limit
       lower="0"
@@ -125,55 +175,55 @@
   </joint>
   <link
-    name="front-left-wheeel">
-    <inertial>
-      <origin
-        xyz="-0.00757015271891448 2.77555756156289E-17 -0.0758230359970678"
-        rpy="0 0 0" />
-      <mass
-        value="2.43249992415545" />
-      <inertia
-        ixx="0.00760381168766053"
-        ixy="-8.24720643585744E-19"
-        ixz="0.00051389219741489"
-        iyy="0.00755250482076537"
-        iyz="-3.62054828260286E-19"
-        izz="0.0126996752980334" />
-    </inertial>
-    <visual>
-      <origin
-        xyz="0 0 0"
-        rpy="0 0 0" />
-      <geometry>
-        <mesh
-          filename="package://car_robot/meshes/front-left-wheeel.STL" />
-      </geometry>
-      <material
-        name="">
-        <color
-          rgba="0 0 0 1" />
-      </material>
-    </visual>
-    <collision>
-      <origin
-        xyz="0 0 0"
-        rpy="0 0 0" />
-      <geometry>
-        <mesh
-          filename="package://car_robot/meshes/front-left-wheeel.STL" />
-      </geometry>
-    </collision>
-  </link>
-  <joint
-    name="fl-wheel"
-    type="revolute">
-    <origin
-      xyz="0.0075702 -0.075823 -0.2005"
-      rpy="1.5708 0 0" />
+    name="front-left-axle">
+    <inertial>
+      <origin
+        xyz="0.00622369727134719 -5.55111512312578E-17 -0.0759454119237932"
+        rpy="0 0 0" />
+      <mass
+        value="0.0772222198144586" />
+      <inertia
+        ixx="0.000151599574572288"
+        ixy="4.39662991317288E-21"
+        ixz="1.19131785081697E-05"
+        iyy="0.000152575854964957"
+        iyz="-5.36504034940161E-20"
+        izz="7.203866309606E-06" />
+    </inertial>
+    <visual>
+      <origin
+        xyz="0 0 0"
+        rpy="0 0 0" />
+      <geometry>
+        <mesh
+          filename="package://car_robot/meshes/front-left-axle.STL" />
+      </geometry>
+      <material
+        name="">
+        <color
+          rgba="0.792156862745098 0.819607843137255 0.933333333333333 1" />
+      </material>
+    </visual>
+    <collision>
+      <origin
+        xyz="0 0 0"
+        rpy="0 0 0" />
+      <geometry>
+        <mesh
+          filename="package://car_robot/meshes/front-left-axle.STL" />
+      </geometry>
+    </collision>
+  </link>
+  <joint
+    name="fl-axle"
+    type="fixed">
+    <origin
+      xyz="-0.00622369727134681 -0.0759454119237924 -0.2005"
+      rpy="1.5707963267949 0 0" />
     <parent
       link="front-left-hinge" />
     <child
-      link="front-left-wheeel" />
-    <axis
-      xyz="0.099346 0 0.99505" />
+      link="front-left-axle" />
+    <axis
+      xyz="-0.0816758172092811 0 0.996658949131144" />
     <limit
       lower="0"
@@ -183,55 +233,113 @@
   </joint>
   <link
-    name="front-left-axle">
-    <inertial>
-      <origin
-        xyz="-0.00757015271891331 -2.77555756156289E-17 -0.0758230359970657"
-        rpy="0 0 0" />
-      <mass
-        value="0.0772222198144586" />
-      <inertia
-        ixx="0.000151131456795402"
-        ixy="-2.82674264757069E-21"
-        ixz="-1.44671657852651E-05"
-        iyy="0.000152575854964957"
-        iyz="-2.83127986289767E-20"
-        izz="7.67198408649241E-06" />
-    </inertial>
-    <visual>
-      <origin
-        xyz="0 0 0"
-        rpy="0 0 0" />
-      <geometry>
-        <mesh
-          filename="package://car_robot/meshes/front-left-axle.STL" />
-      </geometry>
-      <material
-        name="">
-        <color
-          rgba="0.792156862745098 0.819607843137255 0.933333333333333 1" />
-      </material>
-    </visual>
-    <collision>
-      <origin
-        xyz="0 0 0"
-        rpy="0 0 0" />
-      <geometry>
-        <mesh
-          filename="package://car_robot/meshes/front-left-axle.STL" />
-      </geometry>
-    </collision>
-  </link>
-  <joint
-    name="fl-axle"
-    type="revolute">
-    <origin
-      xyz="0.0075702 -0.075823 -0.2005"
-      rpy="1.5708 0 0" />
-    <parent
-      link="front-left-hinge" />
-    <child
-      link="front-left-axle" />
-    <axis
-      xyz="0.099346 0 0.99505" />
+    name="front-right-hinge">
+    <inertial>
+      <origin
+        xyz="0 -1.38777878078145E-16 -0.118799628145585"
+        rpy="0 0 0" />
+      <mass
+        value="0.633612488698205" />
+      <inertia
+        ixx="0.00421634076613872"
+        ixy="1.97169687775791E-19"
+        ixz="3.34139793073233E-19"
+        iyy="0.00245975887674748"
+        iyz="-4.58614596323022E-19"
+        izz="0.00202629416547586" />
+    </inertial>
+    <visual>
+      <origin
+        xyz="0 0 0"
+        rpy="0 0 0" />
+      <geometry>
+        <mesh
+          filename="package://car_robot/meshes/front-right-hinge.STL" />
+      </geometry>
+      <material
+        name="">
+        <color
+          rgba="1 1 0 1" />
+      </material>
+    </visual>
+    <collision>
+      <origin
+        xyz="0 0 0"
+        rpy="0 0 0" />
+      <geometry>
+        <mesh
+          filename="package://car_robot/meshes/front-right-hinge.STL" />
+      </geometry>
+    </collision>
+  </link>
+  <joint
+    name="fr-hinge"
+    type="continuous">
+    <origin
+      xyz="0.254 -0.1397 0.0608"
+      rpy="0 0 -3.1416" />
+    <parent
+      link="base_link" />
+    <child
+      link="front-right-hinge" />
+    <axis
+      xyz="0 0 -1" />
+    <limit
+      lower="-0.69"
+      upper="0.69"
+      effort="0"
+      velocity="0" />
+  </joint>
+  <link
+    name="front-right-wheel">
+    <inertial>
+      <origin
+        xyz="0 2.77555756156289E-17 -0.0762"
+        rpy="0 0 0" />
+      <mass
+        value="2.43249992415545" />
+      <inertia
+        ixx="0.00755250482076537"
+        ixy="-1.41203303983048E-19"
+        ixz="1.30750629116003E-18"
+        iyy="0.00755250482076537"
+        iyz="-3.76415922197689E-18"
+        izz="0.0127509821649285" />
+    </inertial>
+    <visual>
+      <origin
+        xyz="0 0 0"
+        rpy="0 0 0" />
+      <geometry>
+        <mesh
+          filename="package://car_robot/meshes/front-right-wheel.STL" />
+      </geometry>
+      <material
+        name="">
+        <color
+          rgba="0 0 0 1" />
+      </material>
+    </visual>
+    <collision>
+      <origin
+        xyz="0 0 0"
+        rpy="0 0 0" />
+      <geometry>
+        <mesh
+          filename="package://car_robot/meshes/front-right-wheel.STL" />
+      </geometry>
+    </collision>
+  </link>
+  <joint
+    name="fr-wheel"
+    type="continuous">
+    <origin
+      xyz="0 0.0761999999999998 -0.2005"
+      rpy="1.5707963267949 0 3.14159265358979" />
+    <parent
+      link="front-right-hinge" />
+    <child
+      link="front-right-wheel" />
+    <axis
+      xyz="0 0 -1" />
     <limit
       lower="0"
@@ -241,55 +349,55 @@
   </joint>
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