Commit message: Fixed axle probelem

File: car_robot/urdf/car_robot.urdf.xacro (robot description, xacro)
@@ -5,22 +5,9 @@
 <robot
   name="car_robot" xmlns:xacro="http://ros.org/wiki/xacro">
-  <xacro:macro name="body_color">
-    <visual>
-    <material>
-        <ambient>0.8 0.558823529411765 0.1 1</ambient>
-        <diffuse>0.8 0.558823529411765 0.1 1</diffuse>
-        <specular>0.1 0.1 0.1 1</specular>
-        <emissive>0 0 0 0</emissive>
-    </material>
-    </visual>
-</xacro:macro>
-<gazebo reference="base_link">
-    <xacro:body_color />
-</gazebo>
   <link
     name="base_link">
     <inertial>
       <origin
-        xyz="-0.00677096096599197 -7.40324229928916E-09 0.0650709573527417"
+        xyz="-0.00677096096599193 -7.40324228051496E-09 0.0650709573527417"
         rpy="0 0 0" />
       <mass
@@ -28,8 +15,8 @@
       <inertia
         ixx="1.26922453974044"
-        ixy="1.04912166639753E-07"
+        ixy="1.04912166627371E-07"
         ixz="-0.0347492884684778"
         iyy="3.34453299992272"
-        iyz="1.6440457327724E-08"
+        iyz="1.64404574516637E-08"
         izz="4.11157029873108" />
     </inertial>
@@ -62,14 +49,14 @@
     <inertial>
       <origin
-        xyz="0 2.77555756156289E-17 -0.118799628145585"
-        rpy="0 0 0" />
-      <mass
-        value="0.633612488698204" />
-      <inertia
-        ixx="0.0042046227153009"
-        ixy="-0.000142990919869844"
-        ixz="-1.30495243379754E-18"
-        iyy="0.00247147692758528"
-        iyz="-6.30427138270604E-19"
+        xyz="0 0 -0.118799628145585"
+        rpy="0 0 0" />
+      <mass
+        value="0.633612488698205" />
+      <inertia
+        ixx="0.00421598497152854"
+        ixy="2.499711540899E-05"
+        ixz="-1.35033902121542E-18"
+        iyy="0.00246011467135765"
+        iyz="2.20234865744933E-19"
         izz="0.00202629416547586" />
     </inertial>
@@ -100,5 +87,5 @@
   <joint
     name="fl-hinge"
-    type="continuous">
+    type="revolute">
     <origin
       xyz="0.254 0.1397 0.0608"
@@ -111,6 +98,6 @@
       xyz="0 0 -1" />
     <limit
-      lower="-0.69"
-      upper="0.69"
+      lower="-3.14"
+      upper="3.14"
       effort="0"
       velocity="0" />
@@ -120,15 +107,15 @@
     <inertial>
       <origin
-        xyz="0.00622369727134658 -2.77555756156289E-16 -0.0759454119237928"
+        xyz="0.00108447726862249 1.11022302462516E-16 0.0761922824769925"
         rpy="0 0 0" />
       <mass
         value="2.43249992415545" />
       <inertia
-        ixx="0.00758718354662836"
-        ixy="-1.26731196831282E-18"
-        ixz="-0.000423171308923178"
+        ixx="0.00755355776923952"
+        ixy="1.88640504073853E-18"
+        ixz="7.39771592248954E-05"
         iyy="0.00755250482076537"
-        iyz="-1.68232117058127E-19"
-        izz="0.0127163034390655" />
+        iyz="1.95246869510358E-18"
+        izz="0.0127499292164544" />
     </inertial>
     <visual>
@@ -160,5 +147,5 @@
     type="continuous">
     <origin
-      xyz="-0.00622369727134681 -0.0759454119237924 -0.2005"
+      xyz="-0.00108447726862265 0.0761922824769925 -0.2005"
       rpy="1.5707963267949 0 0" />
     <parent
@@ -167,5 +154,5 @@
       link="front-left-wheeel" />
     <axis
-      xyz="-0.0816758172092811 0 0.996658949131144" />
+      xyz="-0.0142319851525261 0 -0.999898720170507" />
     <limit
       lower="0"
@@ -175,124 +162,66 @@
   </joint>
   <link
-    name="front-left-axle">
-    <inertial>
-      <origin
-        xyz="0.00622369727134719 -5.55111512312578E-17 -0.0759454119237932"
-        rpy="0 0 0" />
-      <mass
-        value="0.0772222198144586" />
-      <inertia
-        ixx="0.000151599574572288"
-        ixy="4.39662991317288E-21"
-        ixz="1.19131785081697E-05"
-        iyy="0.000152575854964957"
-        iyz="-5.36504034940161E-20"
-        izz="7.203866309606E-06" />
-    </inertial>
-    <visual>
-      <origin
-        xyz="0 0 0"
-        rpy="0 0 0" />
-      <geometry>
-        <mesh
-          filename="package://car_robot/meshes/front-left-axle.STL" />
-      </geometry>
-      <material
-        name="">
-        <color
-          rgba="0.792156862745098 0.819607843137255 0.933333333333333 1" />
-      </material>
-    </visual>
-    <collision>
-      <origin
-        xyz="0 0 0"
-        rpy="0 0 0" />
-      <geometry>
-        <mesh
-          filename="package://car_robot/meshes/front-left-axle.STL" />
-      </geometry>
-    </collision>
-  </link>
-  <joint
-    name="fl-axle"
-    type="fixed">
-    <origin
-      xyz="-0.00622369727134681 -0.0759454119237924 -0.2005"
-      rpy="1.5707963267949 0 0" />
-    <parent
-      link="front-left-hinge" />
-    <child
-      link="front-left-axle" />
-    <axis
-      xyz="-0.0816758172092811 0 0.996658949131144" />
+    name="front-right-hinge">
+    <inertial>
+      <origin
+        xyz="-5.55111512312578E-17 -5.55111512312578E-17 -0.118799628145585"
+        rpy="0 0 0" />
+      <mass
+        value="0.633612488698205" />
+      <inertia
+        ixx="0.00421634076613872"
+        ixy="3.80852095203232E-19"
+        ixz="1.69567032741007E-18"
+        iyy="0.00245975887674748"
+        iyz="9.55878885787063E-19"
+        izz="0.00202629416547586" />
+    </inertial>
+    <visual>
+      <origin
+        xyz="0 0 0"
+        rpy="0 0 0" />
+      <geometry>
+        <mesh
+          filename="package://car_robot/meshes/front-right-hinge.STL" />
+      </geometry>
+      <material
+        name="">
+        <color
+          rgba="1 1 0 1" />
+      </material>
+    </visual>
+    <collision>
+      <origin
+        xyz="0 0 0"
+        rpy="0 0 0" />
+      <geometry>
+        <mesh
+          filename="package://car_robot/meshes/front-right-hinge.STL" />
+      </geometry>
+    </collision>
+  </link>
+  <joint
+    name="fr-hinge"
+    type="revolute">
+    <origin
+      xyz="0.254 -0.1397 0.0608"
+      rpy="0 0 -3.1416" />
+    <parent
+      link="base_link" />
+    <child
+      link="front-right-hinge" />
+    <axis
+      xyz="0 0 -1" />
     <limit
-      lower="0"
-      upper="0"
+      lower="-3.14"
+      upper="3.14"
       effort="0"
       velocity="0" />
   </joint>
   <link
-    name="front-right-hinge">
-    <inertial>
-      <origin
-        xyz="0 -1.38777878078145E-16 -0.118799628145585"
-        rpy="0 0 0" />
-      <mass
-        value="0.633612488698205" />
-      <inertia
-        ixx="0.00421634076613872"
-        ixy="1.97169687775791E-19"
-        ixz="3.34139793073233E-19"
-        iyy="0.00245975887674748"
-        iyz="-4.58614596323022E-19"
-        izz="0.00202629416547586" />
-    </inertial>
-    <visual>
-      <origin
-        xyz="0 0 0"
-        rpy="0 0 0" />
-      <geometry>
-        <mesh
-          filename="package://car_robot/meshes/front-right-hinge.STL" />
-      </geometry>
-      <material
-        name="">
-        <color
-          rgba="1 1 0 1" />
-      </material>
-    </visual>
-    <collision>
-      <origin
-        xyz="0 0 0"
-        rpy="0 0 0" />
-      <geometry>
-        <mesh
-          filename="package://car_robot/meshes/front-right-hinge.STL" />
-      </geometry>
-    </collision>
-  </link>
-  <joint
-    name="fr-hinge"
-    type="continuous">
-    <origin
-      xyz="0.254 -0.1397 0.0608"
-      rpy="0 0 -3.1416" />
-    <parent
-      link="base_link" />
-    <child
-      link="front-right-hinge" />
-    <axis
-      xyz="0 0 -1" />
-    <limit
-      lower="-0.69"
-      upper="0.69"
-      effort="0"
-      velocity="0" />
-  </joint>
-  <link
     name="front-right-wheel">
     <inertial>
       <origin
-        xyz="0 2.77555756156289E-17 -0.0762"
+        xyz="-5.55111512312578E-17 0 -0.0762"
         rpy="0 0 0" />
       <mass
@@ -300,8 +229,8 @@
       <inertia
         ixx="0.00755250482076537"
-        ixy="-1.41203303983048E-19"
-        ixz="1.30750629116003E-18"
+        ixy="6.00508507818468E-19"
+        ixz="8.35496005193151E-19"
         iyy="0.00755250482076537"
-        iyz="-3.76415922197689E-18"
+        iyz="-3.98615026528919E-18"
         izz="0.0127509821649285" />
     </inertial>
@@ -334,5 +263,5 @@
     type="continuous">
     <origin
-      xyz="0 0.0761999999999998 -0.2005"
+      xyz="0 0.0761999999999999 -0.2005"
       rpy="1.5707963267949 0 3.14159265358979" />
     <parent
@@ -349,55 +278,108 @@
   </joint>
   <link
-    name="front-right-axle">
-    <inertial>
-      <origin
-        xyz="0 5.55111512312578E-17 -0.0762"
-        rpy="0 0 0" />
-      <mass
-        value="0.0772222198144586" />
-      <inertia
-        ixx="0.000152575854964957"
-        ixy="7.03302044017091E-22"
-        ixz="-2.70384489878801E-22"
-        iyy="0.000152575854964957"
-        iyz="9.66801247676817E-20"
-        izz="6.22758591693701E-06" />
-    </inertial>
-    <visual>
-      <origin
-        xyz="0 0 0"
-        rpy="0 0 0" />
-      <geometry>
-        <mesh
-          filename="package://car_robot/meshes/front-right-axle.STL" />
-      </geometry>
-      <material
-        name="">
-        <color
-          rgba="0.792156862745098 0.819607843137255 0.933333333333333 1" />
-      </material>
-    </visual>
-    <collision>
-      <origin
-        xyz="0 0 0"
-        rpy="0 0 0" />
-      <geometry>
-        <mesh
-          filename="package://car_robot/meshes/front-right-axle.STL" />
-      </geometry>
-    </collision>
-  </link>
-  <joint
-    name="fr-axle"
+    name="Lidar">
+    <inertial>
+      <origin
+        xyz="0 -1.02751096627556E-17 -0.08905"
+        rpy="0 0 0" />
+      <mass
+        value="0.0902446020272643" />
+      <inertia
+        ixx="0.000242182519707747"
+        ixy="9.5944127796284E-22"
+        ixz="-6.99487317772809E-21"
+        iyy="0.000242182519707747"
+        iyz="-2.72604477775199E-20"
+        izz="7.27777593048873E-06" />
+    </inertial>
+    <visual>
+      <origin
+        xyz="0 0 0"
+        rpy="0 0 0" />
+      <geometry>
+        <mesh
+          filename="package://car_robot/meshes/Lidar.STL" />
+      </geometry>
+      <material
+        name="">
+        <color
+          rgba="0 0 0 1" />
+      </material>
+    </visual>
+    <collision>
+      <origin
+        xyz="0 0 0"
+        rpy="0 0 0" />
+      <geometry>
+        <mesh
+          filename="package://car_robot/meshes/Lidar.STL" />
+      </geometry>
+    </collision>
+  </link>
+  <joint
+    name="l-sensor"
     type="fixed">
     <origin
-      xyz="0 0.0761999999999998 -0.2005"
-      rpy="1.5707963267949 0 3.14159265358979" />
-    <parent
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
Commit message: Fixed teleop issue

File: car_robot/urdf/car_robot.urdf.xacro (robot description, xacro)
@@ -5,4 +5,19 @@
 <robot
   name="car_robot" xmlns:xacro="http://ros.org/wiki/xacro">
+  <xacro:macro name="body_color">
+    <visual>
+    <material>
+        <ambient>0.05375 0.05 0.06625 0.82</ambient>
+        <diffuse>0.18275 0.17 0.22525 0.82</diffuse>
+        <specular>0.332741 0.328634 0.346435 0.82</specular>
+        <emissive>0 0 0 0</emissive>
+    </material>
+    </visual>
+</xacro:macro>
+<gazebo reference="base_link">
+    <xacro:body_color />
+</gazebo>
+  # Add this before base link
+<link name="dummy_link"></link>
   <link
     name="base_link">
@@ -45,4 +60,10 @@
     </collision>
   </link>
+  # Add this after base link
+<joint name="dummy_joint" type="fixed">
+    <origin rpy="0 0 0" xyz="0 0 0" />
+    <parent link="dummy_link"/>
+    <child link="base_link"/>
+</joint>
   <link
     name="front-left-hinge">
@@ -100,6 +121,6 @@
       lower="-3.14"
       upper="3.14"
-      effort="0"
-      velocity="0" />
+      effort="100"
+      velocity="100" />
   </joint>
   <link
@@ -216,6 +237,6 @@
       lower="-3.14"
       upper="3.14"
-      effort="0"
-      velocity="0" />
+      effort="100"
+      velocity="100" />
   </joint>
   <link
@@ -506,3 +527,58 @@
     </plugin>
 </gazebo>
+<gazebo reference="Lidar">
+  <sensor name="lidar" type="ray">
+    <pose>0.0 0.0 0.0 0 0 0</pose>
+    <always_on>true</always_on>
+    <visualize>true</visualize>
+    <update_rate>5</update_rate>
+    <ray>
+      <scan>
+        <horizontal>
+          <samples>360</samples>
+          <resolution>1.00000</resolution>
+          <min_angle>0.000000</min_angle>
+          <max_angle>6.280000</max_angle>
+        </horizontal>
+      </scan>
+      <range>
+        <min>0.120000</min>
+        <max>3.5</max>
+        <resolution>0.015000</resolution>
+      </range>
+      <noise>
+        <type>gaussian</type>
+        <mean>0.0</mean>
+        <stddev>0.01</stddev>
+      </noise>
+    </ray>
+    <plugin name="scan" filename="libgazebo_ros_ray_sensor.so">
+      <ros>
+        <remapping>~/out:=scan</remapping>
+      </ros>
+      <output_type>sensor_msgs/LaserScan</output_type>
+      <frame_name>Lidar</frame_name>
+    </plugin>
+  </sensor>
+  </gazebo>
+  <gazebo reference="base_link">
+  <gravity>true</gravity>
+  <sensor name="imu_sensor" type="imu">
+    <always_on>true</always_on>
+    <update_rate>100</update_rate>
+    <visualize>true</visualize>
+    <topic>__default_topic__</topic>
+    <plugin filename="libgazebo_ros_imu_sensor.so" name="imu_plugin">
+      <topicName>imu</topicName>
+      <bodyName>base_link</bodyName>
+      <updateRateHZ>10.0</updateRateHZ>
+      <gaussianNoise>0.0</gaussianNoise>
+      <xyzOffset>0 0 0</xyzOffset>
+      <rpyOffset>0 0 0</rpyOffset>
+      <frameName>base_link</frameName>
+      <initialOrientationAsReference>false</initialOrientationAsReference>
+    </plugin>
+    <pose>0 0 0 0 0 0</pose>
+  </sensor>
+</gazebo>
 </robot>
